File: avdisplay-cape.kicad_pcb (KiCad board)
At the start: 4 copper layers, 100 x 55 mm, 46 parts, among them J101 P8, J102 P9, J103 VIN1, J104 VIN2, J105 CAN2, J106 CAN1, Q101 PSMN4R3-30BL,118, Q102 PSMN4R3-30BL,118, SW101 Address Selector, SW102 CAN Term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

Commit message: First pass at mcp2518 version
Parts:
- removed R107: 10K, Resistor_SMD:R_0603_1608Metric
- removed U105: TXB0104PW, Package_SO:TSSOP-14_4.4x5mm_P0.65mm
- J105: value CAN2 -> CAN1
- J106: value CAN1 -> CAN2
- JP101: value SolderJumper_2_Open -> WP
- U101: value MCP2515-xSO -> MCP2518FD-xST; footprint Package_SO:SOIC-18W_7.5x11.6mm_P1.27mm -> Package_SO:SOIC-14_3.9x8.7mm_P1.27mm
- U104, U106: value MCP2551-I-SN -> MCP2562-E-SN
- moved C109 19.4 mm to (174.1, 114.8), turned to -90 degrees
- moved C108 14.8 mm to (174.1, 100.0), turned to -90 degrees
- moved C103 3.80 mm to (139.2, 115.3)
- moved C104 3.80 mm to (155.6, 115.4)
- moved Y101 3.80 mm to (147.4, 115.6)
- moved U101 1.55 mm to (145.4, 105.6)
- moved C101 1.42 mm to (138.5, 103.4)
Connections:
- C109 pad 1: SYS_5V -> DC_3.3V
- U101 pad 10: unconnected-(U101-~{RX1BF}-Pad10) -> SCK
- U101 pad 11: unconnected-(U101-~{RX0BF}-Pad11) -> MOSI
- U101 pad 12: CAN_INT -> MISO
- U101 pad 13: SCK -> CAN_CS
- U101 pad 14: MOSI -> DC_3.3V
- U101 pad 4: unconnected-(U101-~{TX0RTS}-Pad4) -> CAN_INT
- U101 pad 5: unconnected-(U101-~{TX1RTS}-Pad5) -> Net-(U101-OSC2)
- U101 pad 6: unconnected-(U101-~{TX2RTS}-Pad6) -> Net-(U101-OSC1)
- U101 pad 7: Net-(U101-OSC2) -> GND
- U101 pad 8: Net-(U101-OSC1) -> unconnected-(U101-~{INT1}/GPIO1-Pad8)
- U101 pad 9: GND -> unconnected-(U101-~{INT0}/GPIO0/XSTBY-Pad9)
- U104 pad 1: Net-(U104-TXD) -> DCAN1_TX
- U104 pad 4: Net-(U104-RXD) -> DCAN1_RX
- U104 pad 5: unconnected-(U104-Vref-Pad5) -> DC_3.3V
- U106 pad 1: Net-(U105-B3) -> MCP_CAN_TX
- U106 pad 4: Net-(U105-B4) -> MCP_CAN_RX
- U106 pad 5: unconnected-(U106-Vref-Pad5) -> DC_3.3V
Routing:
- net DC_3.3V: track 36.8 -> 64.8 mm, vias 11 -> 9
- net Net-(U105-B4): track 16.8 -> 0.00 mm
- net Net-(U104-TXD): track 13.4 -> 0.00 mm
- net Net-(U101-~{RESET}): track 11.6 -> 0.00 mm
- net DCAN1_RX: track 39.9 -> 49.1 mm
- net MCP_CAN_RX: track 21.5 -> 29.8 mm, vias 0 -> 2
- net Net-(U105-B3): track 7.98 -> 0.00 mm
- net MCP_CAN_TX: track 23.0 -> 30.4 mm, vias 0 -> 2
- net CAN_INT: track 71.8 -> 78.8 mm
- net DCAN1_TX: track 37.3 -> 44.2 mm
- net Net-(U104-RXD): track 6.93 -> 0.00 mm
- net SYS_5V: track 15.7 -> 11.4 mm, vias 3 -> 2
- net GND: track 44.6 -> 43.3 mm, vias 22 -> 21
- net MOSI: track 35.6 -> 35.1 mm
