File: avdisplay-cape.kicad_sch (KiCad schematic)
At the start: 46 parts, among them J101 P8, J102 P9, J103 VIN1, J104 VIN2, J105 CAN2, J106 CAN1, Q101 PSMN4R3-30BL,118, Q102 PSMN4R3-30BL,118, SW101 Address Selector, SW102 CAN Term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

Commit message: First pass at mcp2518 version
Parts:
- removed R107: 10K, Resistor_SMD:R_0603_1608Metric, symbol Device:R
- removed U101: MCP2515-xSO, Package_SO:SOIC-18W_7.5x11.6mm_P1.27mm, symbol Interface_CAN_LIN:MCP2515-xSO
- removed U104, U106: MCP2551-I-SN, Package_SO:SOIC-8_3.9x4.9mm_P1.27mm, symbol Interface_CAN_LIN:MCP2551-I-SN
- removed U105: TXB0104PW, Package_SO:TSSOP-14_4.4x5mm_P0.65mm, symbol Logic_LevelTranslator:TXB0104PW
- added U101: MCP2518FD-xST, Package_SO:SOIC-14_3.9x8.7mm_P1.27mm, symbol Interface_CAN_LIN:MCP2518FD-xQBB
- added U104, U106: MCP2562-E-SN, Package_SO:SOIC-8_3.9x4.9mm_P1.27mm, symbol Interface_CAN_LIN:MCP2562-E-SN
- J105: value CAN2 -> CAN1
- J106: value CAN1 -> CAN2
Connections:
- net +3.3V: now also C109.1, U101.14 (VDD), U104.5 (Vio), U106.5 (Vio)
- net +5V: now also U104.3 (VDD), U106.3 (VDD); no longer C109.1
- net CAN_CS: now also U101.13 (~{CS})
- net CAN_INT: now also U101.4 (~{INT})
- net DCAN1_RX: now also U104.4 (RXD)
- net DCAN1_TX: now also U104.1 (TXD)
- net GND: now also U101.15 (VSS), U101.7 (VSS), U104.2 (VSS), U104.8 (STBY), U106.2 (VSS), U106.8 (STBY)
- net MCP_CAN_RX: now also U101.2 (RXCAN), U106.4 (RXD)
- net MCP_CAN_TX: now also U101.1 (TXCAN), U106.1 (TXD)
- net MISO: now also U101.12 (SDO)
- net MOSI: now also U101.11 (SDI)
- net SCK: now also U101.10 (SCK)
- net at D101.2 (A2), J105.3 (Pin_3), SW102.1: now also U104.6 (CANL)
- net at D102.2 (A2), J106.3 (Pin_3), SW102.2: now also U106.6 (CANL)
- net at D102.1 (A1), J106.2 (Pin_2), R112.2: now also U106.7 (CANH)
- net at D101.1 (A1), J105.2 (Pin_2), R109.1: now also U104.7 (CANH)
- net at C103.1, Y101.1: now also U101.5 (OSC2)
- net at C104.1, Y101.2: now also U101.6 (OSC1)
- no-connect marks 44 -> 39
Other:
- note added: "MCP 2518 CAN FD Controller"
- note removed: "MCP 2515 CAN Controller"
- moved on the sheet: C103, C104, C108, C109, Y101
